File: pcb/imu-beagle-esc-switcheo/imu-beagle-esc-switcheo.sch (KiCad schematic (older format))
At the start: 14 parts, among them K1 CONN_3, K2 CONN_3, K3 CONN_3, P1 CONN_2, P2 CONN_8, P3 CONN_8, P4 CONN_2, P5 CONN_4, P6 CONN_2, P7 CONN_8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

Commit message: un monton de cosas, logs de julio, cosas de la presentacion, kin2z arreglado....
Connections:
- net GND: now also K1.2 (PM); no longer K1.3 (P3)
- net reguladr 11 a 5: no longer K1.2 (PM), P4.1 (P1)
- new net: K1.3 (P3), P4.1 (P1)
Changed lines of the file:
@@
-EESchema Schematic File Version 2  date mar 22 may 2012 18:48:26 UYT
+EESchema Schematic File Version 2  date vie 06 jul 2012 20:10:48 UYT
 LIBS:power
 LIBS:device
@@
 Sheet 1 1
 Title ""
-Date "22 may 2012"
+Date "6 jul 2012"
 Rev ""
 Comp ""
@@
 Comment4 ""
 $EndDescr
+Wire Wire Line
+	4300 1800 6900 1800
+Wire Wire Line
+	4300 1150 3950 1150
+Wire Wire Line
+	3200 1750 3200 2000
+Wire Wire Line
+	3200 1750 3400 1750
+Wire Wire Line
+	2550 1800 2550 2000
+Wire Wire Line
+	2550 2000 3200 2000
+Connection ~ 2800 5550
+Wire Wire Line
+	3250 5550 2800 5550
+Connection ~ 5250 2450
+Wire Wire Line
+	5250 2300 5250 2450
+Connection ~ 5600 1800
+Wire Wire Line
+	5600 1900 5600 1800
+Connection ~ 5600 2850
+Wire Wire Line
+	6900 3100 5600 3100
+Wire Wire Line
+	6900 3100 6900 2850
+Wire Wire Line
+	6900 2850 7150 2850
+Connection ~ 5900 1800
+Wire Wire Line
+	6900 1800 6900 2650
+Wire Wire Line
+	6900 2650 7150 2650
+Connection ~ 4800 2650
+Wire Wire Line
+	4800 2650 4750 2650
+Wire Wire Line
+	4300 2200 4300 2650
+Wire Wire Line
+	4300 2200 4450 2200
+Wire Wire Line
+	4450 2300 3700 2300
+Wire Wire Line
+	3700 2300 3700 2600
+Wire Wire Line
+	2800 2100 4450 2100
+Connection ~ 3550 5200
+Wire Wire Line
+	4300 2650 4850 2650
+Wire Wire Line
+	7250 3550 4750 3550
+Wire Wire Line
+	7250 3550 7250 5750
+Wire Wire Line
+	7250 5750 3550 5750
+Wire Wire Line
+	3550 5750 3550 5100
+Wire Wire Line
+	6400 5150 6500 5150
+Wire Wire Line
+	6500 5050 6400 5050
+Wire Wire Line
+	3700 3300 3700 3950
+Wire Wire Line
+	3700 3950 5900 3950
+Wire Wire Line
+	5900 3950 5900 4850
+Wire Wire Line
+	5900 4850 6500 4850
+Connection ~ 5050 4650
+Connection ~ 4400 3650
+Wire Wire Line
+	3350 3650 5050 3650
+Wire Wire Line
+	5050 3650 5050 4800
+Wire Wire Line
+	5050 5000 4650 5000
+Wire Wire Line
+	4650 5000 4650 4550
+Wire Wire Line
+	4650 4550 6500 4550
+Wire Wire Line
+	3450 5300 3450 3800
+Wire Wire Line
+	3700 2800 3150 2800
+Wire Wire Line
+	3150 2800 3150 4900
+Wire Wire Line
+	3150 4900 3700 4900
+Wire Wire Line
+	4850 2950 4400 2950
+Wire Wire Line
+	4400 2950 4400 3650
+Connection ~ 3350 3650
+Wire Wire Line
+	3700 3200 3350 3200
+Wire Wire Line
+	3350 3200 3350 4700
+Wire Wire Line
+	4850 2850 4650 2850
+Wire Wire Line
+	4650 2850 4650 4250
+Wire Wire Line
+	4650 4250 3700 4250
+Wire Wire Line
+	3700 4250 3700 4600
+Wire Wire Line
+	3350 4700 3700 4700
+Wire Wire Line
+	3250 4800 3700 4800
+Wire Wire Line
+	3700 2900 3250 2900
+Wire Wire Line
+	3700 5000 3050 5000
+Wire Wire Line
+	3050 5000 3050 2700
+Wire Wire Line
+	3050 2700 3700 2700
+Wire Wire Line
+	3450 5300 3700 5300
+Wire Wire Line
+	3450 3800 4500 3800
+Wire Wire Line
+	4500 3800 4500 2750
+Wire Wire Line
+	4500 2750 4850 2750
+Wire Wire Line
+	3700 5200 3550 5200
+Wire Wire Line
+	3550 5100 3700 5100
+Wire Wire Line
+	6500 4650 5050 4650
+Wire Wire Line
+	6500 4750 5800 4750
+Wire Wire Line
+	5800 4750 5800 4050
+Wire Wire Line
+	5800 4050 3250 4050
+Connection ~ 3250 4050
+Wire Wire Line
+	6500 4950 6000 4950
+Wire Wire Line
+	6000 4950 6000 3850
+Wire Wire Line
+	6000 3850 3550 3850
+Wire Wire Line
+	3550 3850 3550 3100
+Wire Wire Line
+	3550 3100 3700 3100
+Wire Wire Line
+	6500 5250 4850 5250
+Wire Wire Line
+	4850 5250 4850 4900
+Wire Wire Line
+	4850 4900 5050 4900
+Wire Wire Line
+	6400 5050 6400 5750
+Connection ~ 6400 5750
+Connection ~ 6400 5150
+Wire Wire Line
+	2800 3850 3350 3850
+Connection ~ 3350 3850
+Connection ~ 2800 3850
+Wire Wire Line
+	3700 3000 2800 3000
+Connection ~ 2800 3000
+Wire Wire Line
+	6150 2650 5900 2650
+Wire Wire Line
+	5900 2650 5900 1800
+Wire Wire Line
+	4750 3550 4750 2450
+Connection ~ 4750 2650
+Wire Wire Line
+	4750 2450 5600 2450
+Wire Wire Line
+	5600 2850 6150 2850
+Wire Wire Line
+	5250 1900 5250 1800
+Connection ~ 5250 1800
+Wire Wire Line
+	5600 3100 5600 2300
+Connection ~ 5600 2450
+Wire Wire Line
+	3250 2900 3250 5150
+Connection ~ 3250 4800
+Wire Wire Line
+	3400 1650 3200 1650
+Wire Wire Line
+	3200 1650 3200 1400
+Wire Wire Line
+	3200 1400 2550 1400
+Wire Wire Line
+	2550 1400 2550 1600
+Wire Wire Line
+	2800 2000 2800 5700
+Connection ~ 2800 2000
+Connection ~ 2800 2100
+Connection ~ 4300 1800
+Wire Wire Line
+	3400 1850 3400 2000
+Wire Wire Line
+	3400 2000 3950 2000
+Wire Wire Line
+	3950 2000 3950 1150
+Wire Wire Line
+	4300 2100 4300 1350
+Connection ~ 4300 2100
 Text Label 4400 1050 0    60   ~ 0
 Alim Beagle
-Connection ~ 4300 1800
-Wire Wire Line
-	4300 1350 4300 1800
-Connection ~ 2800 2100
-Connection ~ 2800 2000
-Wire Wire Line
-	2800 2000 2800 5700
-Wire Wire Line
-	2550 1600 2550 1400
-Wire Wire Line
-	2550 1400 3200 1400
-Wire Wire Line
-	3200 1400 3200 1650
-Wire Wire Line
-	3200 1650 3400 1650
-Connection ~ 3250 4800
-Wire Wire Line
-	3250 5150 3250 2900
-Connection ~ 5600 2450
-Wire Wire Line
-	5600 2300 5600 3100
-Connection ~ 5250 1800
-Wire Wire Line
-	5250 1900 5250 1800
-Wire Wire Line
-	5600 2850 6150 2850
-Wire Wire Line
-	5600 2450 4750 2450
-Connection ~ 4750 2650
-Wire Wire Line
-	4750 2450 4750 3550
-Connection ~ 4100 2100
-Wire Wire Line
-	4100 2100 4100 1800
-Wire Wire Line
-	5900 1800 5900 2650
-Wire Wire Line
-	5900 2650 6150 2650
-Connection ~ 2800 3000
-Wire Wire Line
-	3700 3000 2800 3000
-Connection ~ 2800 3850
-Connection ~ 3350 3850
-Wire Wire Line
-	2800 3850 3350 3850
-Connection ~ 6400 5150
-Connection ~ 6400 5750
-Wire Wire Line
-	6400 5750 6400 5050
-Wire Wire Line
-	5050 4900 4850 4900
-Wire Wire Line
-	4850 4900 4850 5250
-Wire Wire Line
-	4850 5250 6500 5250
-Wire Wire Line
-	3700 3100 3550 3100
-Wire Wire Line
-	3550 3100 3550 3850
-Wire Wire Line
-	3550 3850 6000 3850
-Wire Wire Line
-	6000 3850 6000 4950
-Wire Wire Line
-	6000 4950 6500 4950
-Connection ~ 3250 4050
-Wire Wire Line
-	3250 4050 5800 4050
-Wire Wire Line
-	5800 4050 5800 4750
-Wire Wire Line
-	5800 4750 6500 4750
-Wire Wire Line
-	6500 4650 5050 4650
-Wire Wire Line
-	3700 5100 3550 5100
-Wire Wire Line
-	3700 5200 3550 5200
-Wire Wire Line
-	4850 2750 4500 2750
-Wire Wire Line
-	4500 2750 4500 3800
-Wire Wire Line
-	4500 3800 3450 3800
-Wire Wire Line
-	3700 5300 3450 5300
-Wire Wire Line
-	3700 2700 3050 2700
-Wire Wire Line
-	3050 2700 3050 5000
-Wire Wire Line
-	3050 5000 3700 5000
-Wire Wire Line
-	3250 2900 3700 2900
-Wire Wire Line
-	3250 4800 3700 4800
-Wire Wire Line
-	3700 4700 3350 4700
-Wire Wire Line
-	3700 4600 3700 4250
-Wire Wire Line
-	3700 4250 4650 4250
-Wire Wire Line
-	4650 4250 4650 2850
-Wire Wire Line
-	4650 2850 4850 2850
-Wire Wire Line
-	3350 4700 3350 3200
-Wire Wire Line
-	3350 3200 3700 3200
-Connection ~ 3350 3650
-Wire Wire Line
-	4400 3650 4400 2950
-Wire Wire Line
-	4400 2950 4850 2950
-Wire Wire Line
-	3700 4900 3150 4900
-Wire Wire Line
-	3150 4900 3150 2800
-Wire Wire Line
-	3150 2800 3700 2800
-Wire Wire Line
-	3450 5300 3450 3800
-Wire Wire Line
-	6500 4550 4650 4550
-Wire Wire Line
-	4650 4550 4650 5000
-Wire Wire Line
-	4650 5000 5050 5000
-Wire Wire Line
-	5050 4800 5050 3650
-Wire Wire Line
-	5050 3650 3350 3650
-Connection ~ 4400 3650
-Connection ~ 5050 4650
-Wire Wire Line
-	6500 4850 5900 4850
-Wire Wire Line
-	5900 4850 5900 3950
-Wire Wire Line
-	5900 3950 3700 3950
-Wire Wire Line
-	3700 3950 3700 3300
-Wire Wire Line
-	6400 5050 6500 5050
-Wire Wire Line
-	6400 5150 6500 5150
-Wire Wire Line
-	3550 5100 3550 5750
-Wire Wire Line
-	3550 5750 7250 5750
-Wire Wire Line
-	7250 5750 7250 3550
-Wire Wire Line
-	7250 3550 4750 3550
-Wire Wire Line
-	4850 2650 4300 2650
-Connection ~ 3550 5200
-Wire Wire Line
-	2800 2100 4450 2100
-Wire Wire Line
-	3700 2600 3700 2300
-Wire Wire Line
-	3700 2300 4450 2300
-Wire Wire Line
-	4450 2200 4300 2200
-Wire Wire Line
-	4300 2200 4300 2650
-Wire Wire Line
-	4800 2650 4750 2650
-Connection ~ 4800 2650
-Wire Wire Line
-	7150 2650 6900 2650
-Wire Wire Line
-	6900 2650 6900 1800
-Wire Wire Line
-	6900 1800 4100 1800
-Connection ~ 5900 1800
-Wire Wire Line
-	7150 2850 6900 2850
-Wire Wire Line
-	6900 2850 6900 3100
-Wire Wire Line
-	6900 3100 5600 3100
-Connection ~ 5600 2850
-Wire Wire Line
-	5600 1900 5600 1800
-Connection ~ 5600 1800
-Wire Wire Line
-	5250 2300 5250 2450
-Connection ~ 5250 2450
-Wire Wire Line
-	3250 5550 2800 5550
-Connection ~ 2800 5550
-Wire Wire Line
-	3400 1850 3200 1850
-Wire Wire Line
-	3200 1850 3200 2000
-Wire Wire Line
-	3200 2000 2550 2000
-Wire Wire Line
-	2550 2000 2550 1800
-Wire Wire Line
-	3400 1750 3400 1150
-Wire Wire Line
-	3400 1150 4300 1150
 $Comp
 L CONN_2 P4
